Commit message: Add omni/mecanum kinematics support and mesh switching
- Replace movebase_kinematics_mecan with movebase_kinematics_omni
- Add kinematic_type launch argument to select diff or omni model
- Switch URDF mesh between rover_cad.stl and omni_cad.stl based on kinematic_type
- Extend sim_robot to handle 4-wheel omni inverse kinematics
- Add strafe axis to teleop joystick mapping
- Update configs and READMEs for omni support

File: src/robot_description/src/description/rover_robot.xacro (robot description, xacro)
@@ -6,4 +6,5 @@
   <xacro:arg name="a" default="1.0"/>
   <xacro:arg name="mesh_enabled" default="true"/>
+  <xacro:arg name="mesh_file" default="rover_cad.stl"/>
   <link name="world"/>
   <xacro:macro name="p_instance" params="r g b a">
@@ -24,5 +25,5 @@
             <origin xyz="0.0 0.0 0.0" rpy="1.57 0.0 -1.57"/>
             <geometry>
-              <mesh filename="package://robot_description/meshes/rover_cad.stl"
+              <mesh filename="package://robot_description/meshes/$(arg mesh_file)"
                     scale="0.001 0.001 0.001"/>
             </geometry>
